File: RGB7Segment/RGB7Segment.kicad_sch (KiCad schematic)
At the start: 21 parts, among them J1 Conn_01x02_Socket, J2 Conn_01x02_Socket

Commit message: Rev out to mfger
Other:
- moved on the sheet: C11, C14
Changed lines of the file:
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@@
 	(symbol
 		(lib_id "power:VCC")
-		(at 169.164 30.734 0)
+		(at 146.05 30.48 0)
 		(unit 1)
 		(exclude_from_sim no)
@@
 		(fields_autoplaced yes)
 		(property "Reference" "#PWR0111"
-			(at 169.164 34.544 0)
+			(at 146.05 34.29 0)
 			(effects
 				(font
@@
 		)
 		(property "Value" "VCC"
-			(at 169.164 27.1582 0)
+			(at 146.05 26.9042 0)
 			(effects
 				(font
@@
 		)
 		(property "Footprint" ""
-			(at 169.164 30.734 0)
+			(at 146.05 30.48 0)
 			(effects
 				(font
@@
 		)
 		(property "Datasheet" ""
-			(at 169.164 30.734 0)
+			(at 146.05 30.48 0)
 			(effects
 				(font
@@
 		)
 		(property "Description" ""
-			(at 169.164 30.734 0)
+			(at 146.05 30.48 0)
 			(effects
 				(font
@@
 	(symbol
 		(lib_id "power:VCC")
-		(at 105.41 181.356 0)
+		(at 93.98 92.71 0)
 		(unit 1)
 		(exclude_from_sim no)
@@
 		(fields_autoplaced yes)
 		(property "Reference" "#PWR0152"
-			(at 105.41 185.166 0)
+			(at 93.98 96.52 0)
 			(effects
 				(font
@@
 		)
 		(property "Value" "VCC"
-			(at 105.41 177.7802 0)
+			(at 93.98 89.1342 0)
 			(effects
 				(font
@@
 		)
 		(property "Footprint" ""
-			(at 105.41 181.356 0)
+			(at 93.98 92.71 0)
 			(effects
 				(font
@@
 		)
 		(property "Datasheet" ""
-			(at 105.41 181.356 0)
+			(at 93.98 92.71 0)
 			(effects
 				(font
@@
 		)
 		(property "Description" ""
-			(at 105.41 181.356 0)
+			(at 93.98 92.71 0)
 			(effects
 				(font
@@
 	(symbol
 		(lib_id "Device:C")
-		(at 169.164 34.544 0)
+		(at 146.05 34.29 0)
 		(unit 1)
 		(exclude_from_sim no)
@@
 		(fields_autoplaced yes)
 		(property "Reference" "C11"
-			(at 172.085 33.3318 0)
+			(at 148.971 33.0778 0)
 			(effects
 				(font
@@
 		)
 		(property "Value" "0.1u"
-			(at 172.085 35.7561 0)
+			(at 148.971 35.5021 0)
 			(effects
 				(font
@@
 		)
 		(property "Footprint" "Capacitor_SMD:C_0402_1005Metric"
-			(at 170.1292 38.354 0)
+			(at 147.0152 38.1 0)
 			(effects
 				(font
@@
 		)
 		(property "Datasheet" "~"
-			(at 169.164 34.544 0)
+			(at 146.05 34.29 0)
 			(effects
 				(font
@@
 		)
 		(property "Description" ""
-			(at 169.164 34.544 0)
+			(at 146.05 34.29 0)
 			(effects
 				(font
@@
 	(symbol
 		(lib_id "power:GND")
-		(at 169.164 38.354 0)
+		(at 146.05 38.1 0)
 		(mirror y)
 		(unit 1)
@@
 		(fields_autoplaced yes)
 		(property "Reference" "#PWR0109"
-			(at 169.164 44.704 0)
+			(at 146.05 44.45 0)
 			(effects
 				(font
@@
 		)
 		(property "Value" "GND"
-			(at 169.164 42.7974 0)
+			(at 146.05 42.5434 0)
 			(effects
 				(font
@@
 		)
 		(property "Footprint" ""
-			(at 169.164 38.354 0)
+			(at 146.05 38.1 0)
 			(effects
 				(font
@@
 		)
 		(property "Datasheet" ""
-			(at 169.164 38.354 0)
+			(at 146.05 38.1 0)
 			(effects
 				(font
@@
 		)
 		(property "Description" ""
-			(at 169.164 38.354 0)
+			(at 146.05 38.1 0)
 			(effects
 				(font
@@
 	(symbol
 		(lib_id "power:GND")
-		(at 105.41 188.976 0)
+		(at 93.98 100.33 0)
 		(mirror y)
 		(unit 1)
@@
 		(fields_autoplaced yes)
 		(property "Reference" "#PWR0151"
-			(at 105.41 195.326 0)
+			(at 93.98 106.68 0)
 			(effects
 				(font
@@
 		)
 		(property "Value" "GND"
-			(at 105.41 193.4194 0)
+			(at 93.98 104.7734 0)
 			(effects
 				(font
@@
 		)
 		(property "Footprint" ""
-			(at 105.41 188.976 0)
+			(at 93.98 100.33 0)
 			(effects
 				(font
@@
 		)
 		(property "Datasheet" ""
-			(at 105.41 188.976 0)
+			(at 93.98 100.33 0)
 			(effects
 				(font
@@
 		)
 		(property "Description" ""
-			(at 105.41 188.976 0)
+			(at 93.98 100.33 0)
 			(effects
 				(font
@@
 	(symbol
 		(lib_id "Device:C")
-		(at 105.41 185.166 0)
+		(at 93.98 96.52 0)
 		(unit 1)
 		(exclude_from_sim no)
@@
 		(fields_autoplaced yes)
 		(property "Reference" "C14"
-			(at 108.331 183.9538 0)
+			(at 96.901 95.3078 0)
 			(effects
 				(font
@@
 		)
 		(property "Value" "0.1u"
-			(at 108.331 186.3781 0)
+			(at 96.901 97.7321 0)
 			(effects
 				(font
@@
 		)
 		(property "Footprint" "Capacitor_SMD:C_0402_1005Metric"
-			(at 106.3752 188.976 0)
+			(at 94.9452 100.33 0)
 			(effects
 				(font
@@
 		)
 		(property "Datasheet" "~"
-			(at 105.41 185.166 0)
+			(at 93.98 96.52 0)
 			(effects
 				(font
@@
 		)
 		(property "Description" ""
-			(at 105.41 185.166 0)
+			(at 93.98 96.52 0)
 			(effects
 				(font
